File: mclon_nano_0_1.brd (EAGLE design)
At the start: 53.3 x 68.6 mm, 71 parts, among them J2 10118194-0001LF/C, T1 2N2222, T1.1 BC847, T2 2N2222, T2.1 BC847, U1 TP5400, X1 AK550/2, X2 AK550/2, X3 AK550/2

Commit message: Update img
Other:
- board text added: "ES000027"
Changed lines of the file:
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@@
 <layer number="19" name="Unrouted" color="6" fill="1" visible="yes" active="yes"/>
 <layer number="20" name="Dimension" color="24" fill="1" visible="yes" active="yes"/>
-<layer number="21" name="tPlace" color="7" fill="1" visible="yes" active="yes"/>
-<layer number="22" name="bPlace" color="7" fill="1" visible="no" active="yes"/>
-<layer number="23" name="tOrigins" color="15" fill="1" visible="yes" active="yes"/>
-<layer number="24" name="bOrigins" color="15" fill="1" visible="no" active="yes"/>
-<layer number="25" name="tNames" color="7" fill="1" visible="yes" active="yes"/>
+<layer number="21" name="tPlace" color="7" fill="1" visible="no" active="yes"/>
+<layer number="22" name="bPlace" color="7" fill="1" visible="yes" active="yes"/>
+<layer number="23" name="tOrigins" color="15" fill="1" visible="no" active="yes"/>
+<layer number="24" name="bOrigins" color="15" fill="1" visible="yes" active="yes"/>
+<layer number="25" name="tNames" color="7" fill="1" visible="no" active="yes"/>
 <layer number="26" name="bNames" color="7" fill="1" visible="no" active="yes"/>
-<layer number="27" name="tValues" color="7" fill="1" visible="yes" active="yes"/>
+<layer number="27" name="tValues" color="7" fill="1" visible="no" active="yes"/>
 <layer number="28" name="bValues" color="7" fill="1" visible="no" active="yes"/>
 <layer number="29" name="tStop" color="7" fill="3" visible="no" active="yes"/>
 <layer number="30" name="bStop" color="7" fill="6" visible="no" active="yes"/>
-<layer number="31" name="tCream" color="7" fill="4" visible="yes" active="yes"/>
+<layer number="31" name="tCream" color="7" fill="4" visible="no" active="yes"/>
 <layer number="32" name="bCream" color="7" fill="5" visible="no" active="yes"/>
 <layer number="33" name="tFinish" color="6" fill="3" visible="no" active="yes"/>
@@
 <dimension x1="5.08" y1="0" x2="48.9585" y2="20.1295" x3="67.31" y3="10.06475" textsize="1.778" layer="47" dtype="vertical"/>
 <text x="48.1965" y="55.245" size="1.27" layer="21" font="vector" rot="R180" align="center">XDeSIG</text>
+<text x="30.226" y="29.718" size="1.27" layer="21" font="vector" ratio="13">ES000027</text>
+<text x="39.116" y="29.591" size="1.27" layer="22" font="vector" ratio="13" rot="MR0">ES000027</text>
 </plain>
 <attributes>
