File: electronics/mclon_nano_0_1.brd (EAGLE design)
At the start: 53.3 x 68.6 mm, 71 parts, among them J2 10118194-0001LF/C, T1 2N2222, T1.1 BC847, T2 2N2222, T2.1 BC847, U1 TP5400, X1 AK550/2, X2 AK550/2, X3 AK550/2

Commit message: Update
Parts:
- D2: value SS34 -> 1N5817; device escorna_ELIB:DIODE_SMA -> adafruit:DO35-7
- D2.1: value (none) -> SS34; device adafruit:DO35-7 -> escorna_ELIB:DIODE_SMA
- X1, X2, X3: value AK550/2 -> KF350-2
Changed lines of the file:
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@@
 <attribute name="VALUE" x="38.5191" y="53.0479" size="0.8128" layer="27" font="vector" ratio="10" rot="R90"/>
 </element>
-<element name="X2" library="con-ptr500" package="AK550/2" value="AK550/2" x="47.752" y="5.969" smashed="yes">
+<element name="X2" library="con-ptr500" package="AK550/2" value="KF350-2" x="47.752" y="5.969" smashed="yes">
 <attribute name="OC_NEWARK" value="unknown" x="47.752" y="5.969" size="1.778" layer="27" display="off"/>
 <attribute name="MPN" value="" x="47.752" y="5.969" size="1.778" layer="27" display="off"/>
@@
 <attribute name="OC_FARNELL" value="unknown" x="47.752" y="5.969" size="1.778" layer="27" display="off"/>
 </element>
-<element name="X3" library="con-ptr500" package="AK550/2" value="AK550/2" x="54.737" y="5.969" smashed="yes">
+<element name="X3" library="con-ptr500" package="AK550/2" value="KF350-2" x="54.737" y="5.969" smashed="yes">
 <attribute name="OC_NEWARK" value="unknown" x="54.737" y="5.969" size="1.778" layer="27" display="off"/>
 <attribute name="MPN" value="" x="54.737" y="5.969" size="1.778" layer="27" display="off"/>
@@
 <attribute name="VALUE" x="7.0485" y="35.179" size="0.8128" layer="27" font="vector"/>
 </element>
-<element name="X1" library="con-ptr500" package="AK550/2" value="AK550/2" x="20.5105" y="3.6195" smashed="yes">
+<element name="X1" library="con-ptr500" package="AK550/2" value="KF350-2" x="20.5105" y="3.6195" smashed="yes">
 <attribute name="OC_NEWARK" value="unknown" x="20.5105" y="3.6195" size="1.778" layer="27" display="off"/>
 <attribute name="MPN" value="" x="20.5105" y="3.6195" size="1.778" layer="27" display="off"/>
@@
 <element name="T2.1" library="nxp_60" package="SOT23" value="BC847" x="34.9885" y="49.4665" smashed="yes"/>
 <element name="U$2" library="xdesig" package="OSHW" value="OSHW" x="34.0995" y="33.3375" rot="MR0"/>
-<element name="D2" library="escorna_ELIB" package="DIODE_SMA" value="SS34" x="16.1925" y="13.6525" smashed="yes">
+<element name="D2.1" library="escorna_ELIB" package="DIODE_SMA" value="SS34" x="16.1925" y="13.6525" smashed="yes">
 <attribute name="NAME" x="21.3045" y="14.268" size="0.8128" layer="25" font="vector" ratio="10" rot="R270"/>
 <attribute name="VALUE" x="10.4215" y="14.9665" size="0.8128" layer="27" font="vector" ratio="10" rot="R270"/>
 </element>
-<element name="D2.1" library="adafruit" package="DO35-7" value="" x="16.1925" y="13.6525" smashed="yes">
+<element name="D2" library="adafruit" package="DO35-7" value="1N5817" x="16.1925" y="13.6525" smashed="yes">
 <attribute name="VALUE" x="13.9065" y="10.9855" size="1.27" layer="27" ratio="10"/>
 </element>
@@
 <via x="37.0205" y="45.593" extent="1-16" drill="0.5"/>
 <via x="39.751" y="46.863" extent="1-16" drill="0.5"/>
+<contactref element="D2.1" pad="A"/>
 <contactref element="D2" pad="A"/>
-<contactref element="D2.1" pad="A"/>
 <via x="20.193" y="35.052" extent="1-16" drill="0.5"/>
 <via x="6.9215" y="9.0805" extent="1-16" drill="0.5"/>
@@
 <contactref element="F1" pad="1"/>
 <contactref element="F1.1" pad="1"/>
+<contactref element="D2.1" pad="C"/>
 <contactref element="D2" pad="C"/>
-<contactref element="D2.1" pad="C"/>
 <wire x1="12.3825" y1="13.6525" x2="12.3825" y2="48.514" width="1.4224" layer="16"/>
 <wire x1="12.3825" y1="48.514" x2="14.0335" y2="50.7365" width="1.4224" layer="16"/>
