File: electronics/nClon_001.brd (EAGLE design)
At the start: 53.3 x 68.6 mm, 71 parts, among them J2 10118194-0001LF/C, T1 2N2222, T1.1 BC847, T2 2N2222, T2.1 BC847, U1 TP5400, X1 KF350-2, X2 KF350-2, X3 KF350-2

Commit message: Rename
Parts:
- moved C1 0.57 mm to (47.8, 9.97)
- moved C1.1 0.57 mm to (47.8, 9.97)
- moved C2 0.57 mm to (54.7, 9.97)
- moved C2.1 0.57 mm to (54.7, 9.97)
- moved U$7 0.38 mm to (34.7, 33.3)
Routing:
- net MLY: track 68.6 -> 69.5 mm
Other:
- board text added: "V001 2231"
- board text added: "nClon"
- board text removed: "NanoClon"
- board text removed: "V0.001 2222"
